Commit message: demo

File: caster_description/urdf/caster.urdf.xacro (robot description, xacro)
@@ -22,4 +22,9 @@
         </material>
       </visual>
+      <collision>
+        <geometry>
+          <box size="0.0185 0.0185 0.1338"/>
+        </geometry>
+      </collision>
       <xacro:default_inertial mass="0.1" />
     </link>
@@ -34,5 +39,5 @@
   <xacro:macro name="drive_wheel" params="parent location invert *origin">
     <link name="drive_wheel_${location}_link">
-      <!-- xacro:default_inertial mass="0.1" / -->
+      <xacro:default_inertial mass="0.1" />
       <visual>
         <origin xyz="0 0 0" rpy="0 0 ${invert*M_PI}" />
@@ -81,5 +86,5 @@
   <link name="base_footprint">
     <origin xyz="0 0 0" rpy="0 0 0" />
-    <!-- <xacro:default_inertial mass="0.0001" /> -->
+    <xacro:default_inertial mass="0.0001" />
   </link>
   <!-- base link -->
@@ -94,8 +99,18 @@
       </material>
     </visual>
-    <xacro:default_inertial mass="10" />
+    <collision>
+      <geometry>
+        <box size="0.54 0.54 0.001"/>
+      </geometry>
+    </collision>
+<!--     <collision>
+      <geometry>
+         <cylinder length="0.037" radius="0.27"/>
+      </geometry>
+    </collision> -->
+    <xacro:default_inertial mass="20" />
   </link>
   <joint name="base_link_joint" type="fixed">
-    <origin xyz="0 0 0.030" rpy="0 0 0" />
+    <origin xyz="0 0 0.03" rpy="0 0 0" />
     <parent link="base_footprint" />
     <child link="base_link" />
@@ -109,5 +124,19 @@
   </joint>
   <!-- Laser link -->
-  <link name="laser_link" />
+  <link name="laser_link">
+    <collision>
+      <geometry>
+        <cylinder length="0.0315" radius="0.055"/>
+      </geometry>
+    </collision>
+    <inertial>
+      <!-- <mass value="0.114" /> -->
+      <mass value="0.001" />
+      <origin xyz="0 0 0" />
+      <inertia ixx="0.001" ixy="0.0" ixz="0.0"
+               iyy="0.001" iyz="0.0"
+               izz="0.001" />
+    </inertial>
+  </link>
   <joint name="laser_link_joint" type="fixed">
     <origin xyz="0.2301 0 0.147" rpy="0 0 0" />

File: caster_description/urdf/caster_gazebo.xacro (robot description, xacro)
@@ -24,26 +24,8 @@
         </material>
       </visual>
-<!--     <collision>
-      <geometry>
-         <cylinder length="0.035" radius="0.074"/>
-      </geometry>
-    </collision> -->
-<!--       <collision>
-        <geometry>
-          <box size="0.0185 0.001 0.001"/>
-        </geometry>
-      </collision> -->
       <collision>
         <geometry>
           <box size="0.0185 0.0185 0.1338"/>
         </geometry>
-<!--         <surface>
-          <friction>
-            <ode>
-              <mu>0</mu>
-              <mu2>0</mu2>
-            </ode>
-          </friction>
-        </surface> -->
       </collision>
       <xacro:default_inertial mass="0.1" />
@@ -129,5 +111,5 @@
       </geometry>
     </collision> -->
-    <xacro:default_inertial mass="25" />
+    <xacro:default_inertial mass="20" />
   </link>
   <joint name="base_link_joint" type="fixed">

File: caster_description/urdf/caster_xacro.xacro (robot description, xacro)
@@ -1,8 +1,7 @@
 <?xml version = "1.0"?>
-<robot name = "caster_xacro" xmlns:xacro = "http://www.ros.org/wiki/xacro">
+<robot name = "caster_xacro" xmlns:xacro = "http://ros.org/wiki/xacro">
   <!-- Include accessories -->
   <xacro:include filename = "$(find caster_description)/urdf/common_properties.xacro" />
   <xacro:include filename = "$(find caster_description)/urdf/caster.urdf.xacro" />
   <xacro:include filename = "$(find caster_description)/urdf/iqr_caster.gazebo.xacro" />
-  <xacro:caster/>
 </robot>

File: caster_description/urdf/iqr_caster.gazebo.xacro (robot description, xacro)
@@ -9,8 +9,4 @@
     <turnGravityOff>false</turnGravityOff>
   </gazebo>
-<!--   <gazebo reference="laser_scan_link">
-    <material>Gazebo</material>
-    <turnGravityOff>false</turnGravityOff>
-  </gazebo> -->
   <gazebo reference="support_wheel_front_left_link">
     <material>Gazebo/dark</material>
@@ -69,6 +65,6 @@
       <leftJoint>drive_wheel_left_joint</leftJoint>
       <rightJoint>drive_wheel_right_joint</rightJoint>
-      <wheelSeparation>0.160</wheelSeparation>
-      <wheelDiameter>0.066</wheelDiameter>
+      <wheelSeparation>0.4174</wheelSeparation>
+      <wheelDiameter>0.15</wheelDiameter>
       <wheelAcceleration>1</wheelAcceleration>
       <wheelTorque>10</wheelTorque>
@@ -86,5 +82,5 @@
       <rpyOffset>0 0 0</rpyOffset>
       <updateRateHZ>20.0</updateRateHZ>
-<!--       <imu>
+      <imu>
         <noise>
           <type>gaussian</type>
@@ -102,5 +98,5 @@
           </accel>
         </noise>
-      </imu> -->
+      </imu>
     </plugin>
   </gazebo>
@@ -116,4 +112,5 @@
             <samples>720</samples>
             <resolution>1</resolution>
+            <!-- resolution ???? -->
             <min_angle>0.0</min_angle>
             <max_angle>6.28319</max_angle>

Commit message: demo

File: caster_description/urdf/caster.urdf.xacro (robot description, xacro)
@@ -2,12 +2,4 @@
 <robot name="caster_robot" xmlns:xacro="http://ros.org/wiki/xacro" description="iqr caster robot">
   <xacro:property name="M_PI" value="3.1415926535897931" />
-  <xacro:macro name="default_inertial" params="mass">
-    <inertial>
-      <mass value="${mass}" />
-    <inertia ixx="1.0" ixy="0.0" ixz="0.0"
-             iyy="1.0" iyz="0.0"
-             izz="1.0" />
-    </inertial>
-  </xacro:macro>
   <!-- support_wheel unit -->
   <xacro:macro name="support_wheel" params="parent location *origin">
@@ -27,5 +19,18 @@
         </geometry>
       </collision>
-      <xacro:default_inertial mass="0.1" />
+      <inertial>
+        <origin xyz="0 0 0" />
+        <mass value="0.163" />
+        <inertia ixx="0.1" ixy="0.001" ixz="0.001"
+                 iyy="0.1" iyz="0.001"
+                 izz="0.1" />
+      </inertial>
+      <inertial>
+        <origin xyz="0 0 0" />
+        <mass value="0.163" />
+        <inertia ixx="0.304" ixy="0.001" ixz="-0.126"
+                 iyy="1.45" iyz="0.369"
+                 izz="0.110" />
+      </inertial>
     </link>
     <joint name="support_wheel_${location}_joint" type="fixed">
@@ -39,5 +44,4 @@
   <xacro:macro name="drive_wheel" params="parent location invert *origin">
     <link name="drive_wheel_${location}_link">
-      <xacro:default_inertial mass="0.1" />
       <visual>
         <origin xyz="0 0 0" rpy="0 0 ${invert*M_PI}" />
@@ -55,4 +59,11 @@
         </geometry>
       </collision>
+      <inertial>
+        <origin xyz="0 0 0" />
+        <mass value="0.803" />
+        <inertia ixx="0.0016" ixy="0.0" ixz="-0.0"
+                 iyy="0.003" iyz="0.0"
+                 izz="0.0016" />
+      </inertial>
     </link>
     <joint name="drive_wheel_${location}_joint" type="continuous">
@@ -75,5 +86,11 @@
         </material>
       </visual>
-      <xacro:default_inertial mass="0.1" />
+      <inertial>
+        <origin xyz="0 0 0" />
+        <inertia ixx="0.0" ixy="0.0" ixz="-0.0"
+                 iyy="0.0" iyz="0.0"
+                 izz="0.0" />
+        <mass value="0.01" />
+      </inertial>
     </link>
     <joint name="ultrasonic_${location}_joint" type="fixed">
@@ -86,5 +103,4 @@
   <link name="base_footprint">
     <origin xyz="0 0 0" rpy="0 0 0" />
-    <xacro:default_inertial mass="0.0001" />
   </link>
   <!-- base link -->
@@ -101,13 +117,14 @@
     <collision>
       <geometry>
-        <box size="0.54 0.54 0.001"/>
+         <cylinder length="0.001" radius="0.27"/>
       </geometry>
     </collision>
-<!--     <collision>
-      <geometry>
-         <cylinder length="0.037" radius="0.27"/>
-      </geometry>
-    </collision> -->
-    <xacro:default_inertial mass="20" />
+    <inertial>
+      <origin xyz="0 0 0" />
+      <mass value="42" />
+      <inertia ixx="1.34" ixy="0.016" ixz="0.024"
+               iyy="1.45" iyz="0.006"
+               izz="1.20" />
+    </inertial>
   </link>
   <joint name="base_link_joint" type="fixed">
@@ -131,6 +148,5 @@
     </collision>
     <inertial>
-      <!-- <mass value="0.114" /> -->
-      <mass value="0.001" />
+      <mass value="0.13" />
       <origin xyz="0 0 0" />
       <inertia ixx="0.001" ixy="0.0" ixz="0.0"
@@ -145,5 +161,13 @@
   </joint>
   <!-- Laser link 2 (rplidar) -->
-  <link name="laser_link2" />
+  <link name="laser_link2" >
+    <inertial>
+      <mass value="0.19" />
+      <origin xyz="0 0 0" />
+      <inertia ixx="0.001" ixy="0.0" ixz="0.0"
+               iyy="0.001" iyz="0.0"
+               izz="0.001" />
+    </inertial>
+  </link>
   <joint name="laser_link_joint2" type="fixed">
     <origin xyz="0.01525 0 0.2115" rpy="0 0 ${M_PI}" />

File: caster_description/urdf/caster_gazebo.xacro (robot description, xacro)
@@ -4,12 +4,4 @@
   <xacro:include filename="$(find caster_description)/urdf/iqr_caster.gazebo.xacro"/>
   <xacro:property name="M_PI" value="3.1415926535897931" />
-  <xacro:macro name="default_inertial" params="mass">
-    <inertial>
-      <mass value="${mass}" />
-    <inertia ixx="1.0" ixy="0.0" ixz="0.0"
-             iyy="1.0" iyz="0.0"
-             izz="1.0" />
-    </inertial>
-  </xacro:macro>
   <!-- support_wheel unit -->
   <xacro:macro name="support_wheel" params="parent location *origin">
@@ -29,5 +21,11 @@
         </geometry>
       </collision>
-      <xacro:default_inertial mass="0.1" />
+      <inertial>
+        <origin xyz="0 0 0" />
+        <mass value="0.163" />
+        <inertia ixx="0.304" ixy="0.001" ixz="-0.126"
+                 iyy="1.45" iyz="0.369"
+                 izz="0.110" />
+      </inertial>
     </link>
     <joint name="support_wheel_${location}_joint" type="fixed">
@@ -41,5 +39,4 @@
   <xacro:macro name="drive_wheel" params="parent location invert *origin">
     <link name="drive_wheel_${location}_link">
-      <xacro:default_inertial mass="0.1" />
       <visual>
         <origin xyz="0 0 0" rpy="0 0 ${invert*M_PI}" />
@@ -57,4 +54,11 @@
         </geometry>
       </collision>
+      <inertial>
+        <origin xyz="0 0 0" />
+        <mass value="0.803" />
+        <inertia ixx="0.0016" ixy="0.0" ixz="-0.0"
+                 iyy="0.003" iyz="0.0"
+                 izz="0.0016" />
+      </inertial>
     </link>
     <joint name="drive_wheel_${location}_joint" type="continuous">
@@ -77,5 +81,8 @@
         </material>
       </visual>
-      <xacro:default_inertial mass="0.1" />
+<!--       <inertial>
+        <origin xyz="0 0 0" />
+        <mass value="0.01" />
+      </inertial> -->
     </link>
     <joint name="ultrasonic_${location}_joint" type="fixed">
@@ -88,5 +95,4 @@
   <link name="base_footprint">
     <origin xyz="0 0 0" rpy="0 0 0" />
-    <xacro:default_inertial mass="0.0001" />
   </link>
   <!-- base link -->
@@ -103,13 +109,14 @@
     <collision>
       <geometry>
-        <box size="0.54 0.54 0.001"/>
+         <cylinder length="0.001" radius="0.27"/>
       </geometry>
     </collision>
-<!--     <collision>
-      <geometry>
-         <cylinder length="0.037" radius="0.27"/>
-      </geometry>
-    </collision> -->
-    <xacro:default_inertial mass="20" />
+    <inertial>
+      <origin xyz="0 0 0" />
+      <mass value="42" />
+      <inertia ixx="1.34" ixy="0.016" ixz="0.024"
+               iyy="1.45" iyz="0.006"
+               izz="1.20" />
+    </inertial>
   </link>
   <joint name="base_link_joint" type="fixed">
@@ -127,4 +134,19 @@
   <!-- Laser link -->
   <link name="laser_link">
+    <inertial>
+      <mass value="0.13" />
+      <origin xyz="0 0 0" />
+      <inertia ixx="0.001" ixy="0.0" ixz="0.0"
+               iyy="0.001" iyz="0.0"
+               izz="0.001" />
+    </inertial>
+  </link>
+  <joint name="laser_link_joint" type="fixed">
+    <origin xyz="0.2301 0 0.147" rpy="0 0 0" />
+    <parent link="base_link" />
+    <child link="laser_link" />
+  </joint>
+  <!-- Laser link 2 (rplidar) -->
+  <link name="laser_link2" >
     <collision>
       <geometry>
@@ -133,6 +155,5 @@
     </collision>
     <inertial>
-      <!-- <mass value="0.114" /> -->
-      <mass value="0.001" />
+      <mass value="0.19" />
       <origin xyz="0 0 0" />
       <inertia ixx="0.001" ixy="0.0" ixz="0.0"
@@ -141,11 +162,4 @@
     </inertial>
   </link>
-  <joint name="laser_link_joint" type="fixed">
-    <origin xyz="0.2301 0 0.147" rpy="0 0 0" />
-    <parent link="base_link" />
-    <child link="laser_link" />
-  </joint>
-  <!-- Laser link 2 (rplidar) -->
-  <link name="laser_link2" />
   <joint name="laser_link_joint2" type="fixed">
     <origin xyz="0.01525 0 0.2115" rpy="0 0 ${M_PI}" />

File: caster_description/urdf/iqr_caster.gazebo.xacro (robot description, xacro)
@@ -10,24 +10,46 @@
   </gazebo>
   <gazebo reference="support_wheel_front_left_link">
+    <mu1>0.001</mu1>
+    <mu2>0.001</mu2>
     <material>Gazebo/dark</material>
     <turnGravityOff>false</turnGravityOff>
   </gazebo>
   <gazebo reference="support_wheel_rear_left_link">
+    <mu1>0.001</mu1>
+    <mu2>0.001</mu2>
     <material>Gazebo/dark</material>
     <turnGravityOff>false</turnGravityOff>
   </gazebo>
   <gazebo reference="support_wheel_front_right_link">
+    <mu1>0.001</mu1>
+    <mu2>0.001</mu2>
     <material>Gazebo/dark</material>
     <turnGravityOff>false</turnGravityOff>
   </gazebo>
   <gazebo reference="support_wheel_rear_right_link">
+    <mu1>0.001</mu1>
+    <mu2>0.001</mu2>
     <material>Gazebo/dark</material>
     <turnGravityOff>false</turnGravityOff>
   </gazebo>
   <gazebo reference="drive_wheel_left_link">
+    <mu1>1.0</mu1>
+    <mu2>1.0</mu2>
+    <kp>10000000.0</kp>
+    <kd>1.0</kd>
+    <minDepth>0.001</minDepth>
+    <maxVel>0.1</maxVel>
+    <fdir1>1 0 0</fdir1>
     <material>Gazebo/dark</material>
     <turnGravityOff>false</turnGravityOff>
   </gazebo>
   <gazebo reference="drive_wheel_right_link">
+    <mu1>1.0</mu1>
+    <mu2>1.0</mu2>
+    <kp>10000000.0</kp>
+    <kd>1.0</kd>
+    <minDepth>0.001</minDepth>
+    <maxVel>0.1</maxVel>
+    <fdir1>1 0 0</fdir1>
     <material>Gazebo/dark</material>
     <turnGravityOff>false</turnGravityOff>
@@ -52,4 +74,5 @@
     <plugin name="caster_controller" filename="libgazebo_ros_diff_drive.so">
       <alwaysOn>true</alwaysOn>
+      <!-- <commandTopic>yocs_cmd_vel_mux/input/navigation_cmd</commandTopic> -->
       <commandTopic>cmd_vel</commandTopic>
       <odometryTopic>odom</odometryTopic>
@@ -68,5 +91,5 @@
       <wheelDiameter>0.15</wheelDiameter>
       <wheelAcceleration>1</wheelAcceleration>
-      <wheelTorque>10</wheelTorque>
+      <wheelTorque>6.5</wheelTorque>
       <rosDebugLevel>na</rosDebugLevel>
     </plugin>
@@ -110,13 +133,13 @@
         <scan>
           <horizontal>
-            <samples>720</samples>
-            <resolution>1</resolution>
+            <samples>1080</samples>
+            <resolution>0.25</resolution>
             <!-- resolution ???? -->
             <min_angle>0.0</min_angle>
-            <max_angle>6.28319</max_angle>
+            <max_angle>4.71239</max_angle>
           </horizontal>
         </scan>
         <range>
-          <min>0.120</min>
+          <min>0.06</min>
           <max>20</max>
           <resolution>0.015</resolution>
@@ -134,3 +157,36 @@
     </sensor>
   </gazebo>
+  <gazebo reference="laser_link2">
+    <material>Gazebo/FlatBlack</material>
+    <sensor type="ray" name="lds_lfcd_sensor">
+      <pose>0 0 0 0 0 0</pose>
+      <visualize>false</visualize>
+      <update_rate>10</update_rate>
+      <ray>
+        <scan>
+          <horizontal>
+            <samples>400</samples>
+            <resolution>0.9</resolution>
+            <!-- resolution ???? -->
+            <min_angle>0.0</min_angle>
+            <max_angle>6.28319</max_angle>
+          </horizontal>
+        </scan>
+        <range>
+          <min>0.2</min>
+          <max>8</max>
+          <resolution>0.015</resolution>
+        </range>
+        <noise>
+          <type>gaussian</type>
+          <mean>0.0</mean>
+          <stddev>0.01</stddev>
+        </noise>
+      </ray>
+      <plugin name="gazebo_ros_lds_lfcd_controller" filename="libgazebo_ros_laser.so">
+        <topicName>scan2</topicName>
+        <frameName>laser_link2</frameName>
+      </plugin>
+    </sensor>
+  </gazebo>
 </robot>

Commit message: demo

File: caster_description/urdf/caster.urdf.xacro (robot description, xacro)
@@ -19,11 +19,4 @@
         </geometry>
       </collision>
-      <inertial>
-        <origin xyz="0 0 0" />
-        <mass value="0.163" />
-        <inertia ixx="0.1" ixy="0.001" ixz="0.001"
-                 iyy="0.1" iyz="0.001"
-                 izz="0.1" />
-      </inertial>
       <inertial>
         <origin xyz="0 0 0" />

File: caster_description/urdf/iqr_caster.gazebo.xacro (robot description, xacro)
@@ -2,9 +2,9 @@
 <robot name="caster_sim" xmlns:xacro="http://ros.org/wiki/xacro" description="iqr caster">
   <gazebo reference="footprint">
-    <material>Gazebo/dark</material>
+    <material>Gazebo/Grey</material>
     <turnGravityOff>false</turnGravityOff>
   </gazebo>
   <gazebo reference="base_link">
-    <material>Gazebo/ivory_white</material>
+    <material>Gazebo/Ivory_white</material>
     <turnGravityOff>false</turnGravityOff>
   </gazebo>
@@ -12,5 +12,5 @@
     <mu1>0.001</mu1>
     <mu2>0.001</mu2>
-    <material>Gazebo/dark</material>
+    <material>Gazebo/Grey</material>
     <turnGravityOff>false</turnGravityOff>
   </gazebo>
@@ -18,5 +18,5 @@
     <mu1>0.001</mu1>
     <mu2>0.001</mu2>
-    <material>Gazebo/dark</material>
+    <material>Gazebo/Grey</material>
     <turnGravityOff>false</turnGravityOff>
   </gazebo>
@@ -24,5 +24,5 @@
     <mu1>0.001</mu1>
     <mu2>0.001</mu2>
-    <material>Gazebo/dark</material>
+    <material>Gazebo/Grey</material>
     <turnGravityOff>false</turnGravityOff>
   </gazebo>
@@ -30,5 +30,5 @@
     <mu1>0.001</mu1>
     <mu2>0.001</mu2>
-    <material>Gazebo/dark</material>
+    <material>Gazebo/Grey</material>
     <turnGravityOff>false</turnGravityOff>
   </gazebo>
@@ -41,5 +41,5 @@
     <maxVel>0.1</maxVel>
     <fdir1>1 0 0</fdir1>
-    <material>Gazebo/dark</material>
+    <material>Gazebo/Grey</material>
     <turnGravityOff>false</turnGravityOff>
   </gazebo>
@@ -52,21 +52,21 @@
     <maxVel>0.1</maxVel>
     <fdir1>1 0 0</fdir1>
-    <material>Gazebo/dark</material>
+    <material>Gazebo/Grey</material>
     <turnGravityOff>false</turnGravityOff>
   </gazebo>
   <gazebo reference="ultrasound_front_left_link">
-    <material>Gazebo/dark</material>
+    <material>Gazebo/Grey</material>
     <turnGravityOff>false</turnGravityOff>
   </gazebo>
   <gazebo reference="ultrasound_rear_left_link">
-    <material>Gazebo/dark</material>
+    <material>Gazebo/Grey</material>
     <turnGravityOff>false</turnGravityOff>
   </gazebo>
   <gazebo reference="ultrasound_front_right_link">
-    <material>Gazebo/dark</material>
+    <material>Gazebo/Grey</material>
     <turnGravityOff>false</turnGravityOff>
   </gazebo>
   <gazebo reference="ultrasound_rear_right_link">
-    <material>Gazebo/dark</material>
+    <material>Gazebo/Grey</material>
     <turnGravityOff>false</turnGravityOff>
   </gazebo>
@@ -129,12 +129,12 @@
       <pose>0 0 0 0 0 0</pose>
       <visualize>false</visualize>
-      <update_rate>40</update_rate>
+      <update_rate>20</update_rate>
       <ray>
         <scan>
           <horizontal>
-            <samples>1080</samples>
+            <samples>4320</samples>
             <resolution>0.25</resolution>
             <!-- resolution ???? -->
-            <min_angle>0.0</min_angle>
+            <min_angle>-4.71239</min_angle>
             <max_angle>4.71239</max_angle>
           </horizontal>
@@ -143,5 +143,5 @@
           <min>0.06</min>
           <max>20</max>
-          <resolution>0.015</resolution>
+          <resolution>0.005</resolution>
         </range>
         <noise>
@@ -159,15 +159,15 @@
   <gazebo reference="laser_link2">
     <material>Gazebo/FlatBlack</material>
-    <sensor type="ray" name="lds_lfcd_sensor">
+    <sensor type="ray" name="lds_lfcd_sensor2">
       <pose>0 0 0 0 0 0</pose>
       <visualize>false</visualize>
-      <update_rate>10</update_rate>
+      <update_rate>20</update_rate>
       <ray>
         <scan>
           <horizontal>
-            <samples>400</samples>
+            <samples>800</samples>
             <resolution>0.9</resolution>
             <!-- resolution ???? -->
-            <min_angle>0.0</min_angle>
+            <min_angle>-6.28319</min_angle>
             <max_angle>6.28319</max_angle>
           </horizontal>
@@ -176,5 +176,5 @@
           <min>0.2</min>
           <max>8</max>
-          <resolution>0.015</resolution>
+          <resolution>0.25</resolution>
         </range>
         <noise>
@@ -184,5 +184,5 @@
         </noise>
       </ray>
-      <plugin name="gazebo_ros_lds_lfcd_controller" filename="libgazebo_ros_laser.so">
+      <plugin name="gazebo_ros_lds_lfcd_controller2" filename="libgazebo_ros_laser.so">
         <topicName>scan2</topicName>
         <frameName>laser_link2</frameName>
