Commit message: demo

File: caster_description/urdf/caster.urdf.xacro (robot description, xacro)
@@ -16,5 +16,5 @@
       <collision>
         <geometry>
-          <box size="0.0185 0.0185 0.1338"/>
+          <box size="0.0185 0.0185 0.1335"/>
         </geometry>
       </collision>
@@ -66,4 +66,13 @@
       <axis xyz="0 1 0" rpy="0 0 0"/>
     </joint>
+    <transmission name="tran_${location}">
+      <type>transmission_interface/SimpleTransmission</type>
+      <joint name="drive_wheel_${location}_joint">
+        <hardwareInterface>hardware_interface/VelocityJointInterface</hardwareInterface>
+      </joint>
+      <actuator name="motor_${location}">
+        <mechanicalReduction>1</mechanicalReduction>
+      </actuator>
+    </transmission>
   </xacro:macro>
   <!-- ULT unit-->
@@ -116,5 +125,5 @@
       <origin xyz="0 0 0" />
       <mass value="42" />
-      <inertia ixx="1.34" ixy="0.016" ixz="0.024"
+      <inertia ixx="1.34" ixy="0.016" ixz="-0.024"
                iyy="1.45" iyz="0.006"
                izz="1.20" />

File: caster_description/urdf/iqr_caster.gazebo.xacro (robot description, xacro)
@@ -34,22 +34,8 @@
   </gazebo>
   <gazebo reference="drive_wheel_left_link">
-    <mu1>1.0</mu1>
-    <mu2>1.0</mu2>
-    <kp>10000000.0</kp>
-    <kd>1.0</kd>
-    <minDepth>0.001</minDepth>
-    <maxVel>0.1</maxVel>
-    <fdir1>1 0 0</fdir1>
     <material>Gazebo/Grey</material>
     <turnGravityOff>false</turnGravityOff>
   </gazebo>
   <gazebo reference="drive_wheel_right_link">
-    <mu1>1.0</mu1>
-    <mu2>1.0</mu2>
-    <kp>10000000.0</kp>
-    <kd>1.0</kd>
-    <minDepth>0.001</minDepth>
-    <maxVel>0.1</maxVel>
-    <fdir1>1 0 0</fdir1>
     <material>Gazebo/Grey</material>
     <turnGravityOff>false</turnGravityOff>
@@ -71,28 +57,10 @@
     <turnGravityOff>false</turnGravityOff>
   </gazebo>
-  <gazebo>
-    <plugin name="caster_controller" filename="libgazebo_ros_diff_drive.so">
-      <alwaysOn>true</alwaysOn>
-      <!-- <commandTopic>yocs_cmd_vel_mux/input/navigation_cmd</commandTopic> -->
-      <commandTopic>cmd_vel</commandTopic>
-      <odometryTopic>odom</odometryTopic>
-      <odometryFrame>odom</odometryFrame>
-      <odometrySource>world</odometrySource>
-      <publishOdomTF>true</publishOdomTF>
-      <robotBaseFrame>base_footprint</robotBaseFrame>
-      <publishWheelTF>false</publishWheelTF>
-      <publishTf>true</publishTf>
-      <publishWheelJointState>true</publishWheelJointState>
-      <legacyMode>false</legacyMode>
-      <updateRate>50</updateRate>
-      <leftJoint>drive_wheel_left_joint</leftJoint>
-      <rightJoint>drive_wheel_right_joint</rightJoint>
-      <wheelSeparation>0.4174</wheelSeparation>
-      <wheelDiameter>0.15</wheelDiameter>
-      <wheelAcceleration>1</wheelAcceleration>
-      <wheelTorque>6.5</wheelTorque>
-      <rosDebugLevel>na</rosDebugLevel>
-    </plugin>
-  </gazebo>
+<gazebo>
+  <plugin name="gazebo_ros_control" filename="libgazebo_ros_control.so">
+    <robotNamespace>/</robotNamespace>
+    <legacyModeNS>true</legacyModeNS>
+  </plugin>
+</gazebo>
   <gazebo>
     <plugin name="imu_plugin" filename="libgazebo_ros_imu.so">
@@ -143,5 +111,5 @@
           <min>0.06</min>
           <max>20</max>
-          <resolution>0.005</resolution>
+          <resolution>0.03</resolution>
         </range>
         <noise>
@@ -176,5 +144,5 @@
           <min>0.2</min>
           <max>8</max>
-          <resolution>0.25</resolution>
+          <resolution>0.005</resolution>
         </range>
         <noise>
